File: esp32.kicad_pcb (KiCad board)
At the start: 2 copper layers, 30.5 x 66 mm, 5 parts

Commit message: .
Parts:
- added C1: 1uF/6.3v, PCM_Capacitor_SMD_AKL:C_0603_1608Metric, F.Cu at (166.6, 99.1)
- added C10: 1uF/25v, PCM_Capacitor_SMD_AKL:C_0603_1608Metric, F.Cu at (167.9, 103.6)
- added C2: 0.1uF/16v, PCM_Capacitor_SMD_AKL:C_0603_1608Metric, F.Cu at (168.7, 99.1)
- added C3: 1uF/25v, PCM_Capacitor_SMD_AKL:C_0603_1608Metric, F.Cu at (155.4, 103.6)
- added C4: 1uF/25v, PCM_Capacitor_SMD_AKL:C_0603_1608Metric, F.Cu at (159.5, 103.6)
- added C5: 4.7uF/25v, PCM_Capacitor_SMD_AKL:C_0603_1608Metric, F.Cu at (157.5, 99.8)
- added C6: 1uF/25v, PCM_Capacitor_SMD_AKL:C_0603_1608Metric, F.Cu at (163.6, 103.6)
- added C7: 1uF/25v, PCM_Capacitor_SMD_AKL:C_0603_1608Metric, F.Cu at (161.5, 103.6)
- added C8: 1uF/25v, PCM_Capacitor_SMD_AKL:C_0603_1608Metric, F.Cu at (157.5, 103.6)
- added C9: 1uF/25v, PCM_Capacitor_SMD_AKL:C_0603_1608Metric, F.Cu at (153.4, 103.6)
- added D1: SS2040FL, PCM_Diode_SMD_AKL:D_0603_1608Metric, F.Cu at (154.4, 99.8)
- added D2: SS2040FL, PCM_Diode_SMD_AKL:D_0603_1608Metric, F.Cu at (157.5, 97.5)
- added D3: SS2040FL, PCM_Diode_SMD_AKL:D_0603_1608Metric, F.Cu at (160.5, 99.8)
- added J1: FH34SRJ-24S-0.5SH, custom:FH34SRJ-24S-0.5SH, F.Cu at (164.8, 103.0)
- added L1: L, PCM_Inductor_SMD_AKL:L_1210_3225Metric, F.Cu at (163.6, 98.9)
- added Q2: MCH3478, PCM_Package_TO_SOT_SMD_AKL:SC-59, F.Cu at (171.1, 103.6)
- added R1: 0.47R, PCM_Resistor_SMD_AKL:R_0603_1608Metric, F.Cu at (171.2, 100.3)
Routing:
- net 4: track 0.00 -> 63.1 mm, vias 0 -> 2
- net 3: track 0.00 -> 58.3 mm, vias 0 -> 2
- net 2: track 0.00 -> 53.4 mm, vias 0 -> 2
- net 1: track 0.00 -> 48.7 mm, vias 0 -> 2
- net 10: track 0.00 -> 45.9 mm, vias 0 -> 2
- net 20: track 0.00 -> 43.2 mm, vias 0 -> 2
- net 21: track 0.00 -> 40.5 mm, vias 0 -> 2
- net Net-(D3-A): track 0.00 -> 15.9 mm
- net GND: track 0.00 -> 12.3 mm, vias 0 -> 4
- net Net-(D1-A): track 0.00 -> 10.3 mm
- net Net-(D3-K): track 0.00 -> 8.28 mm
- net Net-(J1-Pin_3): track 0.00 -> 7.73 mm, vias 0 -> 2
- net Net-(J1-Pin_24): track 0.00 -> 7.38 mm
- net +3.3V: track 0.00 -> 6.91 mm, vias 0 -> 3
- net Net-(D1-K): track 0.00 -> 4.86 mm
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Other:
- outline, holes or cut-outs redrawn

Commit message: .
Parts:
- moved C10 115.3 mm to (53.6, 88.4)
- moved C3 115.3 mm to (41.1, 88.4)
- moved C7 115.3 mm to (47.2, 88.4)
- moved J1 115.3 mm to (50.5, 87.7)
- moved Q2 115.3 mm to (56.8, 88.4)
- moved C2 115.3 mm to (54.4, 83.8)
- moved C5 115.3 mm to (43.2, 84.6)
- moved C6 115.3 mm to (49.3, 88.4)
- moved C8 115.3 mm to (43.2, 88.4)
- moved L1 115.3 mm to (49.3, 83.7)
- moved REF** 115.3 mm to (63.5, 99.1)
- moved REF** 115.3 mm to (63.5, 38.1)
- moved REF** 115.3 mm to (38.1, 38.1)
- moved REF** 115.3 mm to (38.1, 99.1)
- moved C1 115.3 mm to (52.3, 83.8)
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Routing:
- net 0: vias 0 -> 1
