File: esp32.kicad_pcb (KiCad board)
At the start: 2 copper layers, 30.5 x 66 mm, 22 parts, among them J1 FH34SRJ-24S-0.5SH, Q2 MCH3478

Commit message: .
Parts:
- added BT1: Battery_Cell, Connector_JST:JST_PH_B2B-PH-SM4-TB_1x02-1MP_P2.00mm_Vertical, F.Cu at (55.4, 64.8)
- added D4: LED, LED_SMD:LED_0603_1608Metric, F.Cu at (46.8, 67.4)
- added Q1: DMG3415U, PCM_Package_TO_SOT_SMD_AKL:SC-59, F.Cu at (48.3, 63.5)
- added R2: 100K, PCM_Resistor_SMD_AKL:R_0603_1608Metric, F.Cu at (48.9, 67.5)
- added R3: 2K (500mA), PCM_Resistor_SMD_AKL:R_0603_1608Metric, F.Cu at (42.8, 67.5)
- added R4: 1K, PCM_Resistor_SMD_AKL:R_0603_1608Metric, F.Cu at (44.8, 67.5)
- added U2: MCP73831-2-OT, Package_TO_SOT_SMD:SOT-23-5, F.Cu at (43.7, 63.5)
Routing:
- net +5V: track 0.00 -> 38.0 mm
- net +BATT: track 0.00 -> 12.9 mm, vias 0 -> 3
- net GND: track 12.7 -> 15.2 mm, vias 4 -> 6
- net Net-(U2-PROG): track 0.00 -> 2.33 mm
- net Net-(U2-STAT): track 0.00 -> 2.23 mm
- net Net-(D4-K): track 0.00 -> 2.06 mm
- net +3.3V: vias 3 -> 4

Commit message: .
Parts:
- L1: value L -> 1276AS-H-100M=P2
- Q2: value MCH3478 -> STR2P3LLH6
- R3: value 2K (500mA) -> 2K
- moved C1 1.52 mm to (53.8, 83.8)
- moved C10 1.52 mm to (55.1, 88.4)
- moved C2 1.52 mm to (55.9, 83.8)
- moved C3 1.52 mm to (44.7, 84.6)
- moved C5 1.52 mm to (48.8, 88.4)
- moved C7 1.52 mm to (44.7, 88.4)
- moved C9 1.52 mm to (40.6, 88.4)
- moved D1 1.52 mm to (41.7, 84.6)
- moved D2 1.52 mm to (44.7, 82.3)
- moved D3 1.52 mm to (47.8, 84.6)
- moved Q2 1.52 mm to (58.4, 88.4)
- moved R1 1.52 mm to (58.9, 85.1)
- moved C4 1.52 mm to (50.8, 88.4)
- moved C6 1.52 mm to (46.7, 88.4)
- moved C8 1.52 mm to (42.7, 88.4)
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- renumbered C5 to C3, C6 to C4, C7 to C5, C4 to C6, C8 to C7, C3 to C8
Routing:
- net +3.3V: track 6.91 -> 9.71 mm, vias 4 -> 6
- net GND: track 15.2 -> 13.2 mm, vias 6 -> 4
- net Net-(J1-Pin_24): track 7.38 -> 5.85 mm
- net Net-(J1-Pin_2): track 4.20 -> 5.67 mm
- net Net-(D1-A): track 10.3 -> 8.93 mm
- net Net-(J1-Pin_20): track 3.33 -> 4.27 mm
- net Net-(J1-Pin_18): track 4.06 -> 4.71 mm
- net Net-(J1-Pin_22): track 4.72 -> 4.10 mm
- net Net-(J1-Pin_3): track 8.11 -> 8.67 mm
- net 0: vias 1 -> 0
Other:
- outline, holes or cut-outs redrawn
- board text added: "C4"
- board text added: "C5"
- board text added: "C6"
- board text added: "C7"
- board text added: "Q1"

Commit message: .
Parts:
- added U3: AP2127N-3.3, Package_TO_SOT_SMD:SOT-23, F.Cu at (50.2, 64.1)
- BT1: footprint Connector_JST:JST_PH_B2B-PH-SM4-TB_1x02-1MP_P2.00mm_Vertical -> Connector_JST:JST_PH_S2B-PH-SM4-TB_1x02-1MP_P2.00mm_Horizontal
- moved Q1 2.58 mm to (45.8, 64.1)
- moved U2 2.47 mm to (41.3, 64.1)
- moved BT1 2.16 mm to (57.0, 66.2), turned to 0 degrees
- moved D4 0.63 mm to (46.6, 68.0)
- moved R3 0.63 mm to (42.6, 68.1)
- moved R2 0.63 mm to (48.7, 68.1)
- moved R4 0.63 mm to (44.6, 68.1)
Connections:
- Q1 pad 2: +3.3V -> Net-(Q1-S)
Routing:
- net Net-(Q1-S): track 0.00 -> 5.09 mm
- net +BATT: track 12.9 -> 15.3 mm
- net +5V: track 38.0 -> 39.8 mm
- net GND: track 13.2 -> 14.3 mm
- net Net-(U2-PROG): track 2.33 -> 3.34 mm
- net Net-(U2-STAT): track 2.23 -> 3.13 mm

Commit message: .
Parts:
- added G***: LOGO, esp32-c3-EPD:zebra, B.Cu at (50.5, 76.5)
- BT1: value Battery_Cell -> S2B-ZR-SM4A-TF
- D4: value LED -> LTST-C191KSKT
- Q1: value DMG3415U -> DMG3415U-7
- U2: value MCP73831-2-OT -> MCP73831T-2ACI/OT
Other:
- board text added: "JLCJLCJLCJLC"
