File: esp32.kicad_sch (KiCad schematic)
At the start: 19 parts, among them J1 FH34SRJ-24S-0.5SH, SW1 SW_Push, SW2 SW_Push

Commit message: .
Parts:
- added Q1: MCH3478, symbol Device:Q_Dual_NMOS_S1G1D2S2G2D1
Connections:
- net at J1.3 (Pin_3), R1.2: now also Q1.1 (S)
- net at C5.1, D3.2 (A), J1.15 (Pin_15)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: now also Q1.6 (D)
- net at J1.2 (Pin_2): now also Q1.2 (G)
Other:
- moved on the sheet: SW1, SW2, U1

Commit message: .
Parts:
- removed Q1: MCH3478, symbol Device:Q_Dual_NMOS_S1G1D2S2G2D1
- removed SW1, SW2: SW_Push, symbol Switch:SW_Push
- added Q2: MCH3478, PCM_Package_TO_SOT_SMD_AKL:SC-59, symbol PCM_Transistor_MOSFET_AKL:Q_NMOS-D_Generic_GDS
- C1, C3, C4, C5, C6, C7: footprint (none) -> PCM_Capacitor_SMD_AKL:C_0603_1608Metric
- C10: renamed from C8; footprint (none) -> PCM_Capacitor_SMD_AKL:C_0603_1608Metric
- C2: value 1uF/16v -> 0.1uF/16v; footprint (none) -> PCM_Capacitor_SMD_AKL:C_0603_1608Metric
- C8: renamed from C9; footprint (none) -> PCM_Capacitor_SMD_AKL:C_0603_1608Metric
- C9: renamed from C10; footprint (none) -> PCM_Capacitor_SMD_AKL:C_0603_1608Metric
- D1, D2, D3: footprint Package_TO_SOT_SMD:TO-252-2_TabPin1 -> PCM_Diode_SMD_AKL:D_0603_1608Metric
- J1: footprint (none) -> custom:FH34SRJ-24S-0.5SH
- L1: footprint (none) -> PCM_Inductor_SMD_AKL:L_1210_3225Metric
- R1: footprint (none) -> PCM_Resistor_SMD_AKL:R_0603_1608Metric
Connections:
- net +3.3V: now also J1.15 (Pin_15), J1.16 (Pin_16)
- net at J1.3 (Pin_3), R1.2: now also Q2.3 (S)
- net at J1.2 (Pin_2): now also Q2.1 (G)
- net at C5.1, D3.2 (A), L1.2: now also Q2.2 (D); no longer J1.15 (Pin_15), J1.16 (Pin_16)
Other:
- moved on the sheet: U1

Commit message: .
Parts:
- added BT1: Battery_Cell, symbol Device:Battery_Cell
- added D4: LED, symbol Device:LED
- added Q1: DMG3415U, Package_TO_SOT_SMD_AKL:SOT-23, symbol PCM_Transistor_MOSFET_AKL:DMG3415U
- added R2: 100K, PCM_Resistor_SMD_AKL:R_0603_1608Metric, symbol Device:R
- added R3: 2K (500mA), PCM_Resistor_SMD_AKL:R_0603_1608Metric, symbol Device:R
- added R4: 1K, PCM_Resistor_SMD_AKL:R_0603_1608Metric, symbol Device:R
- added U2: MCP73831-2-OT, Package_TO_SOT_SMD:SOT-23-5, symbol Battery_Management:MCP73831-2-OT
Connections:
- net +3.3V: now also Q1.2 (S)
- net +5V: now also D4.2 (A), Q1.1 (G), R2.2, U2.4 (V_{DD})
- net GND: now also BT1.2 (-), R2.1, R3.1, U2.2 (V_{SS})
- new net: D4.1 (K), R4.1
- new net: R4.2, U2.1 (STAT)
- new net: R3.2, U2.5 (PROG)
- new net +BATT: BT1.1 (+), Q1.3 (D), U2.3 (V_{BAT})
Other:
- moved on the sheet: C1, C10, C2, C3, C4, C5, C6, C7, C8, C9, D1, D2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

Commit message: .
Parts:
- BT1: footprint (none) -> Connector_JST:JST_PH_B2B-PH-SM4-TB_1x02-1MP_P2.00mm_Vertical
- D4: footprint (none) -> LED_SMD:LED_0603_1608Metric
- Q1: footprint Package_TO_SOT_SMD_AKL:SOT-23 -> PCM_Package_TO_SOT_SMD_AKL:SC-59
Changed lines of the file:
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@@
       (effects (font (size 1.27 1.27)))
     )
-    (property "Footprint" "" (at 149.86 76.2 0)
+    (property "Footprint" "LED_SMD:LED_0603_1608Metric" (at 149.86 76.2 0)
       (effects (font (size 1.27 1.27)) hide)
     )
@@
       (effects (font (size 1.27 1.27)) (justify left))
     )
-    (property "Footprint" "" (at 153.67 50.546 90)
+    (property "Footprint" "Connector_JST:JST_PH_B2B-PH-SM4-TB_1x02-1MP_P2.00mm_Vertical" (at 153.67 50.546 90)
       (effects (font (size 1.27 1.27)) hide)
     )
@@
       (effects (font (size 1.27 1.27)) (justify left))
     )
-    (property "Footprint" "Package_TO_SOT_SMD_AKL:SOT-23" (at 132.08 35.56 0)
-      (effects (font (size 1.27 1.27)) hide)
-    )
+    (property "Footprint" "PCM_Package_TO_SOT_SMD_AKL:SC-59" (at 132.08 35.56 0)
+      (effects (font (size 1.27 1.27)) hide)
+    )

Commit message: .
Parts:
- added U3: AP2127N-3.3, Package_TO_SOT_SMD:SOT-23, symbol Regulator_Linear:AP2127N-3.3
- L1: value L -> 1276AS-H-100M=P2
- Q2: value MCH3478 -> STR2P3LLH6
- R3: value 2K (500mA) -> 2K
- renumbered C5 to C3, C6 to C4, C7 to C5, C4 to C6, C8 to C7, C3 to C8
Connections:
- net +3.3V: now also U3.2 (VO); no longer Q1.2 (S)
- net GND: now also U3.1 (GND)
- new net: Q1.2 (S), U3.3 (VI)
Other:
- moved on the sheet: BT1

Commit message: .
Parts:
- BT1: value Battery_Cell -> S2B-ZR-SM4A-TF; footprint Connector_JST:JST_PH_B2B-PH-SM4-TB_1x02-1MP_P2.00mm_Vertical -> Connector_JST:JST_PH_S2B-PH-SM4-TB_1x02-1MP_P2.00mm_Horizontal
Changed lines of the file:
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@@
       (effects (font (size 1.27 1.27)) (justify left))
     )
-    (property "Value" "Battery_Cell" (at 162.56 56.5785 0)
+    (property "Value" "S2B-ZR-SM4A-TF" (at 162.56 56.5785 0)
       (effects (font (size 1.27 1.27)) (justify left))
     )
-    (property "Footprint" "Connector_JST:JST_PH_B2B-PH-SM4-TB_1x02-1MP_P2.00mm_Vertical" (at 158.75 55.626 90)
+    (property "Footprint" "Connector_JST:JST_PH_S2B-PH-SM4-TB_1x02-1MP_P2.00mm_Horizontal" (at 158.75 55.626 90)
       (effects (font (size 1.27 1.27)) hide)
     )

Commit message: .
Parts:
- D4: value LED -> LTST-C191KSKT
- Q1: value DMG3415U -> DMG3415U-7
- U2: value MCP73831-2-OT -> MCP73831T-2ACI/OT
Changed lines of the file:
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@@
   (symbol (lib_id "Device:LED") (at 149.86 76.2 0) (unit 1)
     (in_bom yes) (on_board yes) (dnp no)
-    (property "Reference" "D4" (at 149.86 81.28 0)
-      (effects (font (size 1.27 1.27)))
-    )
-    (property "Value" "LED" (at 149.86 78.74 0)
+    (property "Reference" "D4" (at 149.86 78.74 0)
+      (effects (font (size 1.27 1.27)))
+    )
+    (property "Value" "LTST-C191KSKT" (at 153.67 81.28 0)
       (effects (font (size 1.27 1.27)))
     )
@@
       (effects (font (size 1.27 1.27)) (justify left))
     )
-    (property "Value" "MCP73831-2-OT" (at 130.4641 66.04 0)
+    (property "Value" "MCP73831T-2ACI/OT" (at 130.4641 66.04 0)
       (effects (font (size 1.27 1.27)) (justify left))
     )
@@
       (effects (font (size 1.27 1.27)) (justify left))
     )
-    (property "Value" "DMG3415U" (at 133.35 39.37 0)
-      (effects (font (size 1.27 1.27)) (justify left))
-    )
+    (property "Value" "DMG3415U-7" (at 133.35 39.37 0)
+      (effects (font (size 1.27 1.27)) (justify left))
+    )
