File: SuperMini-EPD-Sheild.kicad_pcb (KiCad board)
At the start: 2 copper layers, 30.5 x 66 mm, 31 parts, among them J1 FH34SRJ-24S-0.5SH, Q1 DMG3415U-7, Q2 STR2P3LLH6, U2 MCP73831T-2ACI/OT, U3 AP2127N-3.3

Commit message: .
Parts:
- removed the G*** at (50.5, 76.5)
- added G***: LOGO, SuperMini-EPD-Sheild:zebra, F.Cu at (83.3, 68.6)
- added G***: LOGO, SuperMini-EPD-Sheild:zebra, B.Cu at (83.3, 68.6)
- added REF**: MountingHole_2.2mm_M2_Pad, MountingHole:MountingHole_2.2mm_M2_Pad, F.Cu at (70.6, 99.1)
- added REF**: MountingHole_2.2mm_M2_Pad, MountingHole:MountingHole_2.2mm_M2_Pad, F.Cu at (96.0, 38.1)
- added REF**: MountingHole_2.2mm_M2_Pad, MountingHole:MountingHole_2.2mm_M2_Pad, F.Cu at (96.0, 99.1)
- added REF**: MountingHole_2.2mm_M2_Pad, MountingHole:MountingHole_2.2mm_M2_Pad, F.Cu at (70.6, 38.1)
- added mouse-bite-2mm-slot: VAL**, SuperMini-EPD-Sheild:mouse-bite-2mm-slot, F.Cu at (67.1, 40.1)
- added mouse-bite-2mm-slot: VAL**, SuperMini-EPD-Sheild:mouse-bite-2mm-slot, F.Cu at (67.1, 97.0)
Routing:
- added copper zone on B.Cu, net (none)
- added copper zone on F.Cu, net (none)
Other:
- board size 30.5 x 66 mm -> 63 x 66 mm
